File: Gremlin_v3/KiCad/Gremlin_v3/Gremlin_v3.kicad_pcb (KiCad board)
At the start: 2 copper layers, 92 x 112.8 mm, 50 parts, among them J1 JST_02, J2 5034800540, SW1 Switch, SW2 SW_SPST, U1 Nice_Nano_V2

Commit message: Via Holes
Fixed Vias to the correct hole size. Adjusted vias and traces that were affected by the larger via size.
Routing:
- net Net-(J2-Pin_3): track 95.8 -> 101.4 mm
- net Row 2: track 173.2 -> 175.7 mm
- net Net-(J2-Pin_4): track 81.0 -> 82.2 mm
- net Row 0: track 206.0 -> 205.1 mm
- net Net-(J2-Pin_2): track 83.3 -> 84.0 mm
