File: Gremlin_v3/KiCad/Gremlin_v3/Gremlin_v3.kicad_pcb (KiCad board)
At the start: 2 copper layers, 92 x 112.8 mm, 50 parts, among them J1 JST_02, J2 5034800540, SW1 Switch, SW2 SW_SPST, U1 Nice_Nano_V2

Commit message: spring cleaning
Parts:
- added REF**: MountingHole_2.1mm, MountingHole:MountingHole_2.1mm, F.Cu at (108.0, 114.7)
- added REF**: MountingHole_2.1mm, MountingHole:MountingHole_2.1mm, F.Cu at (139.5, 114.3)
- added REF**: MountingHole_2.1mm, MountingHole:MountingHole_2.1mm, F.Cu at (118.5, 148.7)
- added REF**: MountingHole_2.1mm, MountingHole:MountingHole_2.1mm, F.Cu at (117.0, 67.1)
- added REF**: MountingHole_2.1mm, MountingHole:MountingHole_2.1mm, F.Cu at (183.8, 120.7)
- added REF**: MountingHole_2.1mm, MountingHole:MountingHole_2.1mm, F.Cu at (171.6, 56.9)
- added REF**: MountingHole_2.1mm, MountingHole:MountingHole_2.1mm, F.Cu at (135.2, 61.8)

Commit message: Hardware redesign: dedicated screen pads J3, corrected Joy-Con orientation J2, native Col 2 routing, updated firmware overlay, and generated JLCPCB production package
Parts:
- added J3: NiceView_Pads, PinHeader_1x05_P2.54mm_Vertical, F.Cu at (122.0, 115.0)
Connections:
- J2 pad 1: Net-(J2-Pin_1) -> JOY_X
- J2 pad 2: Net-(J2-Pin_2) -> GND
- J2 pad 3: Net-(J2-Pin_3) -> JOY_BTN
- J2 pad 4: Net-(J2-Pin_4) -> JOY_Y
- J2 pad 5: GND -> +3V3
- U1 pad 1: unconnected-(U1-D1-Pad1) -> DISP_CS
- U1 pad 15: unconnected-(U1-D14-Pad15) -> DISP_MOSI
- U1 pad 16: unconnected-(U1-D15-Pad16) -> DISP_SCK
- U1 pad 18: Net-(J2-Pin_3) -> JOY_X
- U1 pad 19: unconnected-(U1-D20-Pad19) -> JOY_Y
- U1 pad 20: Net-(J2-Pin_1) -> JOY_BTN
- U1 pad 21: Net-(J2-Pin_2) -> +3V3
Routing:
- net +3V3: track 0.00 -> 116.7 mm, vias 0 -> 2
- net Net-(J2-Pin_3): track 101.4 -> 0.00 mm, vias 3 -> 0
- net JOY_BTN: track 0.00 -> 96.7 mm, vias 0 -> 2
- net Net-(J2-Pin_2): track 84.0 -> 0.00 mm, vias 2 -> 0
- net Net-(J2-Pin_1): track 83.2 -> 0.00 mm, vias 1 -> 0
- net Net-(J2-Pin_4): track 82.2 -> 0.00 mm, vias 3 -> 0
- net JOY_Y: track 0.00 -> 79.5 mm, vias 0 -> 2
- net JOY_X: track 0.00 -> 76.7 mm
- net DISP_CS: track 0.00 -> 40.9 mm, vias 0 -> 1
- net DISP_SCK: track 0.00 -> 8.84 mm, vias 0 -> 1
- net DISP_MOSI: track 0.00 -> 8.84 mm, vias 0 -> 1
- net Row 3: track 98.4 -> 100.9 mm, vias 4 -> 6
Other:
- board text added: "3V3"
- board text added: "CS"
- board text added: "GND"
- board text added: "MOSI"
- board text added: "NICE!VIEW"
- board text added: "SCK"

Commit message: PCB fixes
Parts:
- removed the REF** at (108.0, 114.7)
