File: Gremlin_v3/KiCad/Gremlin_v3/Gremlin_v3.kicad_sch (KiCad schematic)
At the start: 0 parts

Commit message: Update KiCad Design
Parts:
- added D1, D10, D11, D12, D13, D14, D15, D16, D17, D18, D19, D2, D20, D26, D27, D3, D4, D5, D6, D7, D8, D9: Diode, ScottoKeebs_Components:Diode_SOD-123, symbol scottokeebs:Placeholder_Diode
- added J1: JST_02, Connector_JST:JST_EH_S2B-EH_1x02_P2.50mm_Horizontal, symbol PCM_SL_Connectors:JST_02
- added J2: Conn_01x05, Connector_FFC-FPC:Amphenol_F32Q-1A7x1-11005_1x05-1MP_P0.5mm_Horizontal, symbol Connector_Generic:Conn_01x05
- added S1, S10, S11, S12, S13, S14, S15, S16, S17, S18, S19, S2, S20, S26, S27, S3, S4, S5, S6, S7, S8, S9: Keyswitch, ScottoKeebs_Hotswap:Hotswap_Choc_V1, symbol scottokeebs:Placeholder_Keyswitch
- added SW1: Switch, Button_Switch_SMD:Panasonic_EVQPUJ_EVQPUA, symbol scottokeebs:Placeholder_Switch
- added SW2: SW_SPST, Button_Switch_SMD:SW_SPDT_PCM12, symbol Switch:SW_SPST
- added U1: Nice_Nano_V2, ScottoKeebs_MCU:Nice_Nano_V2, symbol scottokeebs:MCU_Nice_Nano_V2
Connections:
- new net: D9.2 (A), S9.2
- new net: D26.2 (A), S26.2
- new net: D10.2 (A), S10.2
- new net: D8.2 (A), S8.2
- new net: D13.2 (A), S13.2
- new net: D27.2 (A), S27.2
- new net: D4.2 (A), S4.2
- new net: D14.2 (A), S14.2
- new net: D5.2 (A), S5.2
- new net: D16.2 (A), S16.2
- new net: D3.2 (A), S3.2
- new net: D7.2 (A), S7.2
- new net: D11.2 (A), S11.2
- new net: D17.2 (A), S17.2
- new net: D1.2 (A), S1.2
- new net: D20.2 (A), S20.2
- new net: D15.2 (A), S15.2
- new net: D2.2 (A), S2.2
- new net: J1.1, SW2.1 (A)
- new net: J1.2, U1.23 (GND)
- new net: J2.4 (Pin_4), U1.17 (D18)
- new net: J2.3 (Pin_3), U1.18 (D19)
- new net: J2.1 (Pin_1), U1.20 (D21)
- new net: J2.2 (Pin_2), U1.21 (3.3v)
- new net: SW1.2, U1.22 (RST)
- new net: SW2.2 (B), U1.24 (B+)
- new net: J2.5 (Pin_5), SW1.1, U1.3 (GND)
- new net: D18.2 (A), S18.2
- new net: D12.2 (A), S12.2
- new net: D19.2 (A), S19.2
- new net: D6.2 (A), S6.2
- new net Col 0: S1.1, S11.1, S16.1, S6.1, U1.5 (D2)
- new net Col 1: S12.1, S17.1, S2.1, S7.1, U1.6 (D3)
- new net Col 2: S13.1, S18.1, S26.1, S3.1, S8.1, U1.7 (D4)
- new net Col 3: S14.1, S19.1, S27.1, S4.1, S9.1, U1.8 (D5)
- new net Col 4: S10.1, S15.1, S20.1, S5.1, U1.9 (D6)
- new net Row 0: D1.1 (K), D2.1 (K), D3.1 (K), D4.1 (K), D5.1 (K), U1.10 (D7)
- new net Row 1: D10.1 (K), D6.1 (K), D7.1 (K), D8.1 (K), D9.1 (K), U1.11 (D8)
- new net Row 2: D11.1 (K), D12.1 (K), D13.1 (K), D14.1 (K), D15.1 (K), U1.12 (D9)
- new net Row 3: D16.1 (K), D17.1 (K), D18.1 (K), D19.1 (K), D20.1 (K), U1.14 (D16)
- new net Row 4: D26.1 (K), D27.1 (K), U1.13 (D10)
Other:
- title: (none) -> Gremlin v3

Commit message: pcb updates
Parts:
- J2: value Conn_01x05 -> 5034800540; footprint Connector_FFC-FPC:Amphenol_F32Q-1A7x1-11005_1x05-1MP_P0.5mm_Horizontal -> Molex ZIF Connector:CONN_503480-0540_MOL
- renumbered D26 to D21, D27 to D22, S26 to S21, S27 to S22
Changed lines of the file:
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@@
 		(in_pos_files yes)
 		(dnp no)
-		(property "Reference" "D26"
+		(property "Reference" "D21"
 			(at 83.82 151.13 0)
 			(show_name no)
@@
 			(project "Gremlin_v3"
 				(path "/69ac32c3-9673-411f-97e3-71b28a2a4abc"
-					(reference "D26")
+					(reference "D21")
 					(unit 1)
 				)
@@
 		(dnp no)
 		(fields_autoplaced yes)
-		(property "Reference" "S27"
+		(property "Reference" "S22"
 			(at 100.33 137.16 0)
 			(show_name no)
@@
 			(project "Gremlin_v3"
 				(path "/69ac32c3-9673-411f-97e3-71b28a2a4abc"
-					(reference "S27")
+					(reference "S22")
 					(unit 1)
 				)
@@
 		(dnp no)
 		(fields_autoplaced yes)
-		(property "Reference" "S26"
+		(property "Reference" "S21"
 			(at 87.63 137.16 0)
 			(show_name no)
@@
 			(project "Gremlin_v3"
 				(path "/69ac32c3-9673-411f-97e3-71b28a2a4abc"
-					(reference "S26")
+					(reference "S21")
 					(unit 1)
 				)
@@
 			)
 		)
-		(property "Value" "Conn_01x05"
+		(property "Value" "5034800540"
 			(at 240.03 93.98 90)
 			(show_name no)
@@
 			)
 		)
-		(property "Footprint" "Connector_FFC-FPC:Amphenol_F32Q-1A7x1-11005_1x05-1MP_P0.5mm_Horizontal"
+		(property "Footprint" "Molex ZIF Connector:CONN_503480-0540_MOL"
 			(at 240.03 97.79 0)
 			(hide yes)
@@
 		(in_pos_files yes)
 		(dnp no)
-		(property "Reference" "D27"
+		(property "Reference" "D22"
 			(at 96.52 151.13 0)
 			(show_name no)
@@
 			(project "Gremlin_v3"
 				(path "/69ac32c3-9673-411f-97e3-71b28a2a4abc"
-					(reference "D27")
+					(reference "D22")
 					(unit 1)
 				)

Commit message: udpated pcb for cnc
Connections:
- net GND: now reaches J2.5 (Pin_5), SW1.1
- net GND: now also U1.4 (GND); no longer U1.3 (GND)
Changed lines of the file:
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@@
 	)
 	(junction
-		(at 209.55 91.44)
-		(diameter 0)
-		(color 0 0 0 0)
-	)
-	(junction
 		(at 72.39 81.28)
 		(diameter 0)
@@
 	)
 	(junction
+		(at 161.29 97.79)
+		(diameter 0)
+		(color 0 0 0 0)
+	)
+	(junction
 		(at 72.39 101.6)
 		(diameter 0)
@@
 	)
 	(junction
+		(at 163.83 99.06)
+		(diameter 0)
+		(color 0 0 0 0)
+	)
+	(junction
 		(at 85.09 60.96)
 		(diameter 0)
@@
 	(wire
 		(pts
-			(xy 212.09 91.44) (xy 209.55 91.44)
+			(xy 85.09 81.28) (xy 85.09 101.6)
 		)
 		(stroke
@@
 	(wire
 		(pts
-			(xy 85.09 81.28) (xy 85.09 101.6)
+			(xy 201.93 73.66) (xy 201.93 93.98)
 		)
 		(stroke
@@
 	(wire
 		(pts
-			(xy 201.93 73.66) (xy 201.93 93.98)
+			(xy 102.87 73.66) (xy 115.57 73.66)
 		)
 		(stroke
@@
 	(wire
 		(pts
-			(xy 102.87 73.66) (xy 115.57 73.66)
+			(xy 59.69 60.96) (xy 59.69 81.28)
 		)
 		(stroke
@@
 	(wire
 		(pts
-			(xy 59.69 60.96) (xy 59.69 81.28)
+			(xy 90.17 134.62) (xy 102.87 134.62)
 		)
 		(stroke
@@
 	(wire
 		(pts
-			(xy 90.17 134.62) (xy 102.87 134.62)
+			(xy 64.77 114.3) (xy 77.47 114.3)
 		)
 		(stroke
@@
 	(wire
 		(pts
-			(xy 64.77 114.3) (xy 77.47 114.3)
+			(xy 163.83 96.52) (xy 163.83 99.06)
 		)
 		(stroke
@@
 	(wire
 		(pts
+			(xy 209.55 64.77) (xy 161.29 64.77)
+		)
+		(stroke
+			(width 0)
+			(type default)
+		)
+	)
+	(wire
+		(pts
 			(xy 77.47 134.62) (xy 90.17 134.62)
 		)
@@
 	(wire
 		(pts
-			(xy 162.56 96.52) (xy 166.37 96.52)
+			(xy 163.83 99.06) (xy 166.37 99.06)
 		)
 		(stroke
@@
 	(wire
 		(pts
+			(xy 161.29 99.06) (xy 163.83 99.06)
+		)
+		(stroke
+			(width 0)
+			(type default)
+		)
+	)
+	(wire
+		(pts
 			(xy 90.17 154.94) (xy 102.87 154.94)
 		)
@@
 	(wire
 		(pts
+			(xy 209.55 80.01) (xy 209.55 64.77)
+		)
+		(stroke
+			(width 0)
+			(type default)
+		)
+	)
+	(wire
+		(pts
 			(xy 59.69 46.99) (xy 59.69 60.96)
 		)
@@
 	(wire
 		(pts
-			(xy 209.55 91.44) (xy 203.2 91.44)
+			(xy 161.29 97.79) (xy 161.29 99.06)
 		)
 		(stroke
@@
 	(wire
 		(pts
-			(xy 110.49 46.99) (xy 110.49 60.96)
+			(xy 203.2 91.44) (xy 212.09 91.44)
 		)
 		(stroke
@@
 	(wire
 		(pts
-			(xy 102.87 93.98) (xy 115.57 93.98)
+			(xy 110.49 46.99) (xy 110.49 60.96)
 		)
 		(stroke
@@
 	(wire
 		(pts
-			(xy 240.03 106.68) (xy 196.85 106.68)
+			(xy 102.87 93.98) (xy 115.57 93.98)
 		)
 		(stroke
@@
 	(wire
 		(pts
-			(xy 90.17 73.66) (xy 102.87 73.66)
+			(xy 240.03 106.68) (xy 196.85 106.68)
 		)
 		(stroke
@@
 	(wire
 		(pts
-			(xy 237.49 102.87) (xy 237.49 105.41)
+			(xy 90.17 73.66) (xy 102.87 73.66)
 		)
 		(stroke
@@
 	(wire
 		(pts
-			(xy 72.39 46.99) (xy 72.39 60.96)
+			(xy 237.49 102.87) (xy 237.49 105.41)
 		)
 		(stroke
@@
 	(wire
 		(pts
-			(xy 97.79 101.6) (xy 97.79 121.92)
+			(xy 72.39 46.99) (xy 72.39 60.96)
 		)
 		(stroke
@@
 	(wire
 		(pts
-			(xy 199.39 99.06) (xy 196.85 99.06)
+			(xy 97.79 101.6) (xy 97.79 121.92)
 		)
 		(stroke
@@
 	(wire
 		(pts
-			(xy 209.55 80.01) (xy 209.55 91.44)
+			(xy 199.39 99.06) (xy 196.85 99.06)
 		)
 		(stroke
@@
 	(wire
 		(pts
+			(xy 161.29 64.77) (xy 161.29 97.79)
+		)
+		(stroke
+			(width 0)
+			(type default)
+		)
+	)
+	(wire
+		(pts
 			(xy 85.09 101.6) (xy 85.09 121.92)
 		)
@@
 	(wire
 		(pts
+			(xy 162.56 96.52) (xy 163.83 96.52)
+		)
+		(stroke
+			(width 0)
+			(type default)
+		)
+	)
+	(wire
+		(pts
 			(xy 110.49 60.96) (xy 110.49 81.28)
 		)
@@
 	(wire
 		(pts
+			(xy 151.13 97.79) (xy 161.29 97.79)
+		)
+		(stroke
+			(width 0)
+			(type default)
+		)
+	)
+	(wire
+		(pts
 			(xy 190.5 73.66) (xy 201.93 73.66)
 		)
@@
 					(unit 1)
 				)
+			)
+		)
+	)
+	(symbol
+		(lib_id "power:GND")
+		(at 151.13 97.79 0)
+		(unit 1)
+		(body_style 1)
+		(exclude_from_sim no)
+		(in_bom yes)
+		(on_board yes)
+		(in_pos_files yes)
+		(dnp no)
+		(fields_autoplaced yes)
+		(property "Reference" "#PWR01"
+			(at 151.13 104.14 0)
+			(hide yes)
+			(show_name no)
+			(do_not_autoplace no)
+			(effects
+				(font
+					(size 1.27 1.27)
+				)
+			)
+		)
+		(property "Value" "GND"
+			(at 151.13 102.87 0)
+			(show_name no)
+			(do_not_autoplace no)
+			(effects
+				(font
+					(size 1.27 1.27)
+				)
+			)
+		)
+		(property "Footprint" ""
+			(at 151.13 97.79 0)
+			(hide yes)
+			(show_name no)
+			(do_not_autoplace no)
+			(effects
+				(font
+					(size 1.27 1.27)
+				)
+			)
+		)
+		(property "Datasheet" ""
+			(at 151.13 97.79 0)
+			(hide yes)
+			(show_name no)
+			(do_not_autoplace no)
+			(effects
+				(font
+					(size 1.27 1.27)
+				)
+			)
+		)
+		(property "Description" "Power symbol creates a global label with name \"GND\" , ground"
+			(at 151.13 97.79 0)
+			(hide yes)
+			(show_name no)
+			(do_not_autoplace no)
+			(effects
+				(font
+					(size 1.27 1.27)
+				)
+			)
+		)
+		(pin "1"
+		)
+		(instances
+			(project "Gremlin_v3"
+				(path "/69ac32c3-9673-411f-97e3-71b28a2a4abc"
+					(reference "#PWR01")
+					(unit 1)
+				)

Commit message: Hardware redesign: dedicated screen pads J3, corrected Joy-Con orientation J2, native Col 2 routing, updated firmware overlay, and generated JLCPCB production package
Parts:
- added J3: NiceView_Pads, Connector_PinHeader_2.54mm:PinHeader_1x05_P2.54mm_Vertical, symbol Connector_Generic:Conn_01x05
Connections:
- net GND: now also J2.2 (Pin_2), J3.5 (Pin_5); no longer J2.5 (Pin_5)
- net DISP_CS: now reaches U1.1 (D1)
- net DISP_CS: now also J3.1 (Pin_1)
- net DISP_MOSI: now reaches U1.15 (D14)
- net DISP_MOSI: now also J3.3 (Pin_3)
- net DISP_SCK: now reaches U1.16 (D15)
- net DISP_SCK: now also J3.2 (Pin_2)
- net at U1.17 (D18): no longer J2.4 (Pin_4)
- net JOY_BTN: now reaches J2.3 (Pin_3)
- net JOY_BTN: now also U1.20 (D21); no longer U1.18 (D19)
- net JOY_Y: now reaches U1.19 (D20)
- net JOY_Y: now also J2.4 (Pin_4)
- net JOY_X: now reaches J2.1 (Pin_1)
- net JOY_X: now also U1.18 (D19); no longer U1.20 (D21)
- net +3V3: now reaches U1.21 (3.3v)
- net +3V3: now also J2.5 (Pin_5), J3.4 (Pin_4); no longer J2.2 (Pin_2)
